Commit message: Updated generalized model framing

File: src/robot_descriptions/generic_quadruped_description/model/quadruped.urdf (robot description, URDF)
Before this commit: robot quadruped, 18 links, 17 joints
Links:
- link FL_calf: geometry collision box size=0 0 0; visual cylinder length=1 radius=0.1
- link FL_hip: geometry collision box size=0 0 0; visual cylinder length=0.25 radius=0.1
- link FL_thigh: geometry collision box size=0 0 0; visual cylinder length=1 radius=0.1
- link FR_calf: geometry collision box size=0 0 0; visual cylinder length=1 radius=0.1
- link FR_hip: geometry collision box size=0 0 0; visual cylinder length=0.25 radius=0.1
- link FR_thigh: geometry collision box size=0 0 0; visual cylinder length=1 radius=0.1
- link RL_calf: geometry collision box size=0 0 0; visual cylinder length=1 radius=0.1
- link RL_hip: geometry collision box size=0 0 0; visual cylinder length=0.25 radius=0.1
- link RL_thigh: geometry collision box size=0 0 0; visual cylinder length=1 radius=0.1
- link RR_calf: geometry collision box size=0 0 0; visual cylinder length=1 radius=0.1
- link RR_hip: geometry collision box size=0 0 0; visual cylinder length=0.25 radius=0.1
- link RR_thigh: geometry collision box size=0 0 0; visual cylinder length=1 radius=0.1
- link base: geometry collision box size=0 0 0; visual box size=3 2 1
- link base_inertia: geometry collision box size=0 0 0
Joints:
- removed joint FL_foot
- removed joint FR_foot
- removed joint RL_foot
- removed joint RR_foot
- added joint FL_foot_joint: type fixed, parent FL_calf, child FL_foot, origin xyz=1 0 0 rpy=0.0 0.0 0.0
- added joint FR_foot_joint: type fixed, parent FR_calf, child FR_foot, origin xyz=1 0 0 rpy=0.0 0.0 0.0
- added joint RL_foot_joint: type fixed, parent RL_calf, child RL_foot, origin xyz=1 0 0 rpy=0.0 0.0 0.0
- added joint RR_foot_joint: type fixed, parent RR_calf, child RR_foot, origin xyz=1 0 0 rpy=0.0 0.0 0.0
- joint FL_hip_joint: origin xyz=0.5 0.5 0.0 rpy=1.5707963267948966 0.0 1.5707963267948966 -> xyz=1.5 1.0 0.0 rpy=1.5707963267948966 0.0 1.5707963267948966
- joint FR_hip_joint: origin xyz=0.5 -0.5 0.0 rpy=1.5707963267948966 0.0 -1.5707963267948966 -> xyz=1.5 -1.0 0.0 rpy=1.5707963267948966 0.0 -1.5707963267948966
- joint RL_hip_joint: origin xyz=-0.5 0.5 0.0 rpy=1.5707963267948966 0.0 1.5707963267948966 -> xyz=-1.5 1.0 0.0 rpy=1.5707963267948966 0.0 1.5707963267948966
- joint RR_hip_joint: origin xyz=-0.5 -0.5 0.0 rpy=1.5707963267948966 0.0 -1.5707963267948966 -> xyz=-1.5 -1.0 0.0 rpy=1.5707963267948966 0.0 -1.5707963267948966

File: src/robot_descriptions/generic_quadruped_description/xacro/leg.xacro (robot description, xacro)
@@ -3,43 +3,53 @@
     <xacro:include
         filename="/workspace/src/robot_descriptions/generic_quadruped_description/xacro/const.xacro" />
-    <xacro:macro name="base_to_hip_joint" params="name right parent child Px Py Pz roll pitch yaw">
-        <xacro:if value="${right == True}">
-            <joint name="${name}" type="continuous">
+    <xacro:macro name="hip_joint" params="leg_name right Px Py Pz">
+        <joint name="${leg_name}_hip_joint" type="continuous">
+            <parent link="base" />
+            <child link="${leg_name}_hip" />
+            <axis xyz="0 0 1" />
+            <xacro:if value="${right == True}">
                 <origin
                     xyz="${Px} ${Py} ${Pz}"
-                    rpy="${roll+PI/2} ${pitch} ${yaw-PI/2}" />
-                <parent
-                    link="${parent}" />
-                <child
-                    link="${child}" />
-                <axis
-                    xyz="0 0 1" />
-            </joint>
-        </xacro:if>
-        <xacro:if value="${right == False}">
-            <joint name="${name}" type="continuous">
+                    rpy="${PI/2} 0.0 ${-PI/2}" />
+            </xacro:if>
+            <xacro:if value="${right == False}">
                 <origin
                     xyz="${Px} ${Py} ${Pz}"
-                    rpy="${roll+PI/2} ${pitch} ${yaw+PI/2}" />
-                <parent
-                    link="${parent}" />
-                <child
-                    link="${child}" />
-                <axis
-                    xyz="0 0 1" />
-            </joint>
-        </xacro:if>
+                    rpy="${PI/2} 0.0 ${PI/2}" />
+            </xacro:if>
+        </joint>
     </xacro:macro>
-    <xacro:macro name="rev_joint" params="name parent child length roll pitch yaw">
-        <joint name="${name}" type="continuous">
-            <origin
-                xyz="${length} 0 0"
-                rpy="${roll} ${pitch} ${yaw}" />
-            <parent
-                link="${parent}" />
-            <child
-                link="${child}" />
-            <axis
-                xyz="0 0 1" />
+    <xacro:macro name="thigh_joint" params="leg_name right length">
+        <joint name="${leg_name}_thigh_joint" type="continuous">
+            <parent link="${leg_name}_hip" />
+            <child link="${leg_name}_thigh" />
+            <axis xyz="0 0 1" />
+            <xacro:if value="${right == True}">
+                <origin
+                    xyz="${length} 0 0"
+                    rpy="${PI/2} 0.0 ${-PI/2}" />
+            </xacro:if>
+            <xacro:if value="${right == False}">
+                <origin
+                    xyz="${length} 0 0"
+                    rpy="${-PI/2} 0 ${-PI/2}" />
+            </xacro:if>
+        </joint>
+    </xacro:macro>
+    <xacro:macro name="calf_joint" params="leg_name right length">
+        <joint name="${leg_name}_calf_joint" type="continuous">
+            <parent link="${leg_name}_thigh" />
+            <child link="${leg_name}_calf" />
+            <axis xyz="0 0 1" />
+            <xacro:if value="${right == True}">
+                <origin
+                    xyz="${length} 0 0"
+                    rpy="0.0 0.0 0.0" />
+            </xacro:if>
+            <xacro:if value="${right == False}">
+                <origin
+                    xyz="${length} 0 0"
+                    rpy="0.0 0.0 0.0" />
+            </xacro:if>
         </joint>
     </xacro:macro>
@@ -84,5 +94,5 @@
                 </visual>
             </xacro:if>
-            <xacro:no_collision/>
+            <xacro:no_collision />
         </link>
     </xacro:macro>
@@ -111,5 +121,5 @@
                 <material name="grey" />
             </visual>
-            <xacro:no_collision/>
+            <xacro:no_collision />
         </link>
     </xacro:macro>
@@ -157,13 +167,9 @@
     <xacro:macro name="leg" params="leg_name right Px Py Pz rad L1 L2 L3 m1 m2 m3 m4">
         <xacro:link link_name="${leg_name}_hip" mass="${m1}" rad="${rad}" length="${L1}" />
-        <xacro:base_to_hip_joint name="${leg_name}_hip_joint" right="${right}" parent="base"
-            child="${leg_name}_hip"
-            Px="${Px}" Py="${Py}" Pz="${Pz}" roll="0.0" pitch="0.0" yaw="0.0" />
+        <xacro:hip_joint leg_name="${leg_name}" right="${right}" Px="${Px}" Py="${Py}" Pz="${Pz}" />
         <xacro:link link_name="${leg_name}_thigh" mass="${m2}" rad="${rad}" length="${L2}" />
-        <xacro:rev_joint name="${leg_name}_thigh_joint" parent="${leg_name}_hip"
-            child="${leg_name}_thigh" length="${L1}" roll="${PI/2}" pitch="0.0" yaw="${-PI/2}" />
+        <xacro:thigh_joint leg_name="${leg_name}" right="${right}" length="${L1}" />
         <xacro:link link_name="${leg_name}_calf" mass="${m3}" rad="${rad}" length="${L3}" />
-        <xacro:rev_joint name="${leg_name}_calf_joint" parent="${leg_name}_thigh"
-            child="${leg_name}_calf" length="${L2}" roll="0.0" pitch="0.0" yaw="0.0" />
+        <xacro:calf_joint leg_name="${leg_name}" right="${right}" length="${L2}" />
         <xacro:foot foot_name="${leg_name}_foot" mass="${m4}" rad="${rad}" />
         <xacro:fixed_joint name="${leg_name}_foot_joint" parent="${leg_name}_calf"
