Commit message: Confirmed model validity with napkin_calc.py

File: src/quadruped_description/xacro/model.xacro (robot description, xacro)
@@ -4,4 +4,5 @@
         <!-- Robot URDF -->
         <uri>/workspace/install/generic_quadruped_description/share/generic_quadruped_description/model/quadruped.urdf</uri>
+        <!-- <uri>/workspace/src/robot_descriptions/a1_description/urdf/a1.urdf</uri> -->
         <!-- Plugin for joint state publisher -->
         <plugin

File: src/robot_descriptions/generic_quadruped_description/xacro/leg.xacro (robot description, xacro)
@@ -171,4 +171,8 @@
         <xacro:thigh_joint leg_name="${leg_name}" right="${right}" length="${L1}" />
         <xacro:link link_name="${leg_name}_calf" mass="${m3}" rad="${rad}" length="${L3}" />
+        <!-- foot sphere at knee position for contact purposes -->
+        <xacro:foot foot_name="${leg_name}_knee" mass="0.0" rad="${rad}" />
+        <xacro:fixed_joint name="${leg_name}_knee_joint" parent="${leg_name}_calf"
+            child="${leg_name}_knee" length="0.0" />
         <xacro:calf_joint leg_name="${leg_name}" right="${right}" length="${L2}" />
         <xacro:foot foot_name="${leg_name}_foot" mass="${m4}" rad="${rad}" />

File: src/robot_descriptions/generic_quadruped_description/xacro/params.xacro (robot description, xacro)
@@ -9,5 +9,5 @@
     <xacro:property name="FR_rad" value="0.1" />
     <xacro:property name="FR_L1" value="0.25" />
-    <xacro:property name="FR_L2" value="1" />
+    <xacro:property name="FR_L2" value="2" />
     <xacro:property name="FR_L3" value="1" />
     <xacro:property name="FR_m1" value="1" />
