Commit message: Updated quadruped inertia generation

File: src/quadruped_description/xacro/leg.xacro (robot description, xacro)
@@ -65,5 +65,5 @@
         </joint>
     </xacro:macro>
-    <xacro:macro name="base_link" params="name L_x L_y L_z mass inertial_link">
+    <xacro:macro name="base_link" params="name L_x L_y L_z mass inertial_link Ixx Iyy Izz">
         <link name="${name}">
             <xacro:if value="${inertial_link == True}">
@@ -75,10 +75,10 @@
                         value="${mass}" />
                     <inertia
-                        ixx="${(mass / 12) * (L_y*L_y + L_z*L_z)}"
+                        ixx="${Ixx}"
                         ixy="0"
                         ixz="0"
-                        iyy="${(mass / 12) * (L_x*L_x + L_z*L_z)}"
+                        iyy="${Iyy}"
                         iyz="0"
-                        izz="${(mass / 12) * (L_x*L_x + L_y*L_y)}" />
+                        izz="${Izz}" />
                 </inertial>
             </xacro:if>
@@ -97,5 +97,5 @@
         </link>
     </xacro:macro>
-    <xacro:macro name="link" params="link_name mass rad length">
+    <xacro:macro name="link" params="link_name mass rad length Ixx Iyy Izz">
         <link name="${link_name}">
             <inertial>
@@ -105,10 +105,10 @@
                 <mass value="${mass}" />
                 <inertia
-                    ixx="${.5 * mass * rad*rad}"
+                    ixx="${Ixx}"
                     ixy="0"
                     ixz="0"
-                    iyy="${(1/12) * (length*length + 3*rad*rad) * mass}"
+                    iyy="${Iyy}"
                     iyz="0"
-                    izz="${(1/12) * (length*length + 3*rad*rad) * mass}" />
+                    izz="${Izz}" />
             </inertial>
             <visual>
@@ -124,5 +124,5 @@
         </link>
     </xacro:macro>
-    <xacro:macro name="foot" params="foot_name mass rad">
+    <xacro:macro name="foot" params="foot_name mass rad Ixx Iyy Izz">
         <link name="${foot_name}">
             <inertial>
@@ -132,10 +132,10 @@
                 <mass value="${mass}" />
                 <inertia
-                    ixx="${(2/5) * (mass*rad*rad)}"
+                    ixx="${Ixx}"
                     ixy="0"
                     ixz="0"
-                    iyy="${(83/320) * (mass*rad*rad)}"
+                    iyy="${Iyy}"
                     iyz="0"
-                    izz="${(83/320) * (mass*rad*rad)}" />
+                    izz="${Izz}" />
             </inertial>
             <visual>
@@ -165,16 +165,22 @@
         </collision>
     </xacro:macro>
-    <xacro:macro name="leg" params="leg_name right Px Py Pz rad L1 L2 L3 m1 m2 m3 m4">
-        <xacro:link link_name="${leg_name}_hip" mass="${m1}" rad="${rad}" length="${L1}" />
+    <xacro:macro name="leg"
+        params="leg_name right Px Py Pz rad L1 L2 L3 m1 m2 m3 m4 I1xx I1yy I1zz I2xx I2yy I2zz I3xx I3yy I3zz I4xx I4yy I4zz">
+        <xacro:link link_name="${leg_name}_hip" mass="${m1}" rad="${rad}" length="${L1}"
+            Ixx="${I1xx}" Iyy="${I1yy}" Izz="${I1zz}" />
         <xacro:hip_joint leg_name="${leg_name}" right="${right}" Px="${Px}" Py="${Py}" Pz="${Pz}" />
-        <xacro:link link_name="${leg_name}_thigh" mass="${m2}" rad="${rad}" length="${L2}" />
+        <xacro:link link_name="${leg_name}_thigh" mass="${m2}" rad="${rad}" length="${L2}"
+            Ixx="${I2xx}" Iyy="${I2yy}" Izz="${I2zz}" />
         <xacro:thigh_joint leg_name="${leg_name}" right="${right}" length="${L1}" />
-        <xacro:link link_name="${leg_name}_calf" mass="${m3}" rad="${rad}" length="${L3}" />
+        <xacro:link link_name="${leg_name}_calf" mass="${m3}" rad="${rad}" length="${L3}"
+            Ixx="${I3xx}" Iyy="${I3yy}" Izz="${I3zz}" />
         <!-- foot sphere at knee position for contact purposes -->
-        <xacro:foot foot_name="${leg_name}_knee" mass="0.0" rad="${rad}" />
+        <xacro:foot foot_name="${leg_name}_knee" mass="0.0" rad="${rad}"
+            Ixx="${0.0}" Iyy="${0.0}" Izz="${0.0}" />
         <xacro:fixed_joint name="${leg_name}_knee_joint" parent="${leg_name}_calf"
             child="${leg_name}_knee" length="0.0" />
         <xacro:calf_joint leg_name="${leg_name}" right="${right}" length="${L2}" />
-        <xacro:foot foot_name="${leg_name}_foot" mass="${m4}" rad="${rad}" />
+        <xacro:foot foot_name="${leg_name}_foot" mass="${m4}" rad="${rad}"
+            Ixx="${I4xx}" Iyy="${I4yy}" Izz="${I4zz}" />
         <xacro:fixed_joint name="${leg_name}_foot_joint" parent="${leg_name}_calf"
             child="${leg_name}_foot" length="${L3}" />

File: src/quadruped_description/xacro/params.xacro (robot description, xacro)
@@ -1,6 +1,7 @@
 <?xml version="1.0" encoding="utf-8"?>
-<robot name="quadruped" xmlns:xacro="http://www.ros.org/wiki/xacro">
-    <xacro:property name="yaml_file" value="/workspace/src/quadruped_description/config/params.yaml"/>
-    <xacro:property name="quad" value="${xacro.load_yaml(yaml_file)}"/>
+<robot name="quadruped_params" xmlns:xacro="http://www.ros.org/wiki/xacro">
+    <xacro:property name="yaml_file"
+        value="/workspace/build/quadruped_description/config/params.yaml" />
+    <xacro:property name="quad" value="${xacro.load_yaml(yaml_file)}" />
     <!-- Base Parameters -->
     <xacro:property name="base_Lx" value="${quad.base.Lx}" />
@@ -8,4 +9,7 @@
     <xacro:property name="base_Lz" value="${quad.base.Lz}" />
     <xacro:property name="base_m" value="${quad.base.m}" />
+    <xacro:property name="base_Ixx" value="${quad.base.I.Ixx}" />
+    <xacro:property name="base_Iyy" value="${quad.base.I.Iyy}" />
+    <xacro:property name="base_Izz" value="${quad.base.I.Izz}" />
     <!-- FR Leg Parameters -->
     <xacro:property name="FR_rad" value="${quad.FR.rad}" />
@@ -17,4 +21,16 @@
     <xacro:property name="FR_m3" value="${quad.FR.m3}" />
     <xacro:property name="FR_m4" value="${quad.FR.m4}" />
+    <xacro:property name="FR_I1xx" value="${quad.FR.I1.Ixx}" />
+    <xacro:property name="FR_I1yy" value="${quad.FR.I1.Iyy}" />
+    <xacro:property name="FR_I1zz" value="${quad.FR.I1.Izz}" />
+    <xacro:property name="FR_I2xx" value="${quad.FR.I2.Ixx}" />
+    <xacro:property name="FR_I2yy" value="${quad.FR.I2.Iyy}" />
+    <xacro:property name="FR_I2zz" value="${quad.FR.I2.Izz}" />
+    <xacro:property name="FR_I3xx" value="${quad.FR.I3.Ixx}" />
+    <xacro:property name="FR_I3yy" value="${quad.FR.I3.Iyy}" />
+    <xacro:property name="FR_I3zz" value="${quad.FR.I3.Izz}" />
+    <xacro:property name="FR_I4xx" value="${quad.FR.I4.Ixx}" />
+    <xacro:property name="FR_I4yy" value="${quad.FR.I4.Iyy}" />
+    <xacro:property name="FR_I4zz" value="${quad.FR.I4.Izz}" />
     <!-- FL Leg Parameters -->
     <xacro:property name="FL_rad" value="${quad.FL.rad}" />
@@ -26,4 +42,16 @@
     <xacro:property name="FL_m3" value="${quad.FL.m3}" />
     <xacro:property name="FL_m4" value="${quad.FL.m4}" />
+    <xacro:property name="FL_I1xx" value="${quad.FL.I1.Ixx}" />
+    <xacro:property name="FL_I1yy" value="${quad.FL.I1.Iyy}" />
+    <xacro:property name="FL_I1zz" value="${quad.FL.I1.Izz}" />
+    <xacro:property name="FL_I2xx" value="${quad.FL.I2.Ixx}" />
+    <xacro:property name="FL_I2yy" value="${quad.FL.I2.Iyy}" />
+    <xacro:property name="FL_I2zz" value="${quad.FL.I2.Izz}" />
+    <xacro:property name="FL_I3xx" value="${quad.FL.I3.Ixx}" />
+    <xacro:property name="FL_I3yy" value="${quad.FL.I3.Iyy}" />
+    <xacro:property name="FL_I3zz" value="${quad.FL.I3.Izz}" />
+    <xacro:property name="FL_I4xx" value="${quad.FL.I4.Ixx}" />
+    <xacro:property name="FL_I4yy" value="${quad.FL.I4.Iyy}" />
+    <xacro:property name="FL_I4zz" value="${quad.FL.I4.Izz}" />
     <!-- RL Leg Parameters -->
     <xacro:property name="RL_rad" value="${quad.RL.rad}" />
@@ -35,4 +63,16 @@
     <xacro:property name="RL_m3" value="${quad.RL.m3}" />
     <xacro:property name="RL_m4" value="${quad.RL.m4}" />
+    <xacro:property name="RL_I1xx" value="${quad.RL.I1.Ixx}" />
+    <xacro:property name="RL_I1yy" value="${quad.RL.I1.Iyy}" />
+    <xacro:property name="RL_I1zz" value="${quad.RL.I1.Izz}" />
+    <xacro:property name="RL_I2xx" value="${quad.RL.I2.Ixx}" />
+    <xacro:property name="RL_I2yy" value="${quad.RL.I2.Iyy}" />
+    <xacro:property name="RL_I2zz" value="${quad.RL.I2.Izz}" />
+    <xacro:property name="RL_I3xx" value="${quad.RL.I3.Ixx}" />
+    <xacro:property name="RL_I3yy" value="${quad.RL.I3.Iyy}" />
+    <xacro:property name="RL_I3zz" value="${quad.RL.I3.Izz}" />
+    <xacro:property name="RL_I4xx" value="${quad.RL.I4.Ixx}" />
+    <xacro:property name="RL_I4yy" value="${quad.RL.I4.Iyy}" />
+    <xacro:property name="RL_I4zz" value="${quad.RL.I4.Izz}" />
     <!-- RR Leg Parameters -->
     <xacro:property name="RR_rad" value="${quad.RR.rad}" />
@@ -44,3 +84,15 @@
     <xacro:property name="RR_m3" value="${quad.RR.m3}" />
     <xacro:property name="RR_m4" value="${quad.RR.m4}" />
+    <xacro:property name="RR_I1xx" value="${quad.RR.I1.Ixx}" />
+    <xacro:property name="RR_I1yy" value="${quad.RR.I1.Iyy}" />
+    <xacro:property name="RR_I1zz" value="${quad.RR.I1.Izz}" />
+    <xacro:property name="RR_I2xx" value="${quad.RR.I2.Ixx}" />
+    <xacro:property name="RR_I2yy" value="${quad.RR.I2.Iyy}" />
+    <xacro:property name="RR_I2zz" value="${quad.RR.I2.Izz}" />
+    <xacro:property name="RR_I3xx" value="${quad.RR.I3.Ixx}" />
+    <xacro:property name="RR_I3yy" value="${quad.RR.I3.Iyy}" />
+    <xacro:property name="RR_I3zz" value="${quad.RR.I3.Izz}" />
+    <xacro:property name="RR_I4xx" value="${quad.RR.I4.Ixx}" />
+    <xacro:property name="RR_I4yy" value="${quad.RR.I4.Iyy}" />
+    <xacro:property name="RR_I4zz" value="${quad.RR.I4.Izz}" />
 </robot>

File: src/quadruped_description/xacro/quadruped.xacro (robot description, xacro)
@@ -12,21 +12,41 @@
     <xacro:base_link
         name="base" L_x="${base_Lx}" L_y="${base_Ly}" L_z="${base_Lz}" mass="${base_m}"
-        inertial_link="False" />
+        inertial_link="False" Ixx="${base_Ixx}" Iyy="${base_Iyy}" Izz="${base_Izz}"/>
     <!-- Insert dummy link to carry inertia values for base link -->
     <xacro:base_link
         name="base_inertia" L_x="${base_Lx}" L_y="${base_Ly}" L_z="${base_Lz}" mass="${base_m}"
-        inertial_link="True" />
+        inertial_link="True" Ixx="${base_Ixx}" Iyy="${base_Iyy}" Izz="${base_Izz}"/>
     <xacro:fixed_joint name="inertial_base_joint" parent="base" child="base_inertia" length="0.0" />
     <xacro:leg leg_name="FR" right="True"
-        Px="${base_Lx/2}" Py="${-base_Ly/2}" Pz="0.0" rad="${FR_rad}" L1="${FR_L1}" L2="${FR_L2}"
-        L3="${FR_L3}" m1="${FR_m1}" m2="${FR_m2}" m3="${FR_m3}" m4="${FR_m4}" />
+        Px="${base_Lx/2}" Py="${-base_Ly/2}" Pz="0.0" rad="${FR_rad}"
+        L1="${FR_L1}" L2="${FR_L2}" L3="${FR_L3}"
+        m1="${FR_m1}" m2="${FR_m2}" m3="${FR_m3}" m4="${FR_m4}"
+        I1xx="${FR_I1xx}" I1yy="${FR_I1yy}" I1zz="${FR_I1zz}"
+        I2xx="${FR_I2xx}" I2yy="${FR_I2yy}" I2zz="${FR_I2yy}"
+        I3xx="${FR_I3xx}" I3yy="${FR_I3yy}" I3zz="${FR_I3yy}"
+        I4xx="${FR_I4xx}" I4yy="${FR_I4yy}" I4zz="${FR_I4yy}" />
     <xacro:leg leg_name="FL" right="False"
-        Px="${base_Lx/2}" Py="${base_Ly/2}" Pz="0.0" rad="${FL_rad}" L1="${FL_L1}" L2="${FL_L2}"
-        L3="${FL_L3}" m1="${FL_m1}" m2="${FL_m2}" m3="${FL_m3}" m4="${FL_m4}" />
+        Px="${base_Lx/2}" Py="${base_Ly/2}" Pz="0.0" rad="${FL_rad}"
+        L1="${FL_L1}" L2="${FL_L2}" L3="${FL_L3}"
+        m1="${FL_m1}" m2="${FL_m2}" m3="${FL_m3}" m4="${FL_m4}"
+        I1xx="${FL_I1xx}" I1yy="${FL_I1yy}" I1zz="${FL_I1zz}"
+        I2xx="${FL_I2xx}" I2yy="${FL_I2yy}" I2zz="${FL_I2yy}"
+        I3xx="${FL_I3xx}" I3yy="${FL_I3yy}" I3zz="${FL_I3yy}"
+        I4xx="${FL_I4xx}" I4yy="${FL_I4yy}" I4zz="${FL_I4yy}" />
     <xacro:leg leg_name="RL" right="False"
-        Px="${-base_Lx/2}" Py="${base_Ly/2}" Pz="0.0" rad="${RL_rad}" L1="${RL_L1}" L2="${RL_L2}"
-        L3="${RL_L3}" m1="${RL_m1}" m2="${RL_m2}" m3="${RL_m3}" m4="${RL_m4}" />
+        Px="${-base_Lx/2}" Py="${base_Ly/2}" Pz="0.0" rad="${RL_rad}"
+        L1="${RL_L1}" L2="${RL_L2}" L3="${RL_L3}"
+        m1="${RL_m1}" m2="${RL_m2}" m3="${RL_m3}" m4="${RL_m4}"
+        I1xx="${RL_I1xx}" I1yy="${RL_I1yy}" I1zz="${RL_I1zz}"
+        I2xx="${RL_I2xx}" I2yy="${RL_I2yy}" I2zz="${RL_I2yy}"
+        I3xx="${RL_I3xx}" I3yy="${RL_I3yy}" I3zz="${RL_I3yy}"
+        I4xx="${RL_I4xx}" I4yy="${RL_I4yy}" I4zz="${RL_I4yy}" />
     <xacro:leg leg_name="RR" right="True"
-        Px="${-base_Lx/2}" Py="${-base_Ly/2}" Pz="0.0" rad="${RR_rad}" L1="${RR_L1}" L2="${RR_L2}"
-        L3="${RR_L3}" m1="${RR_m1}" m2="${RR_m2}" m3="${RR_m3}" m4="${RR_m4}" />
+        Px="${-base_Lx/2}" Py="${-base_Ly/2}" Pz="0.0" rad="${RR_rad}"
+        L1="${RR_L1}" L2="${RR_L2}" L3="${RR_L3}"
+        m1="${RR_m1}" m2="${RR_m2}" m3="${RR_m3}" m4="${RR_m4}"
+        I1xx="${RR_I1xx}" I1yy="${RR_I1yy}" I1zz="${RR_I1zz}"
+        I2xx="${RR_I2xx}" I2yy="${RR_I2yy}" I2zz="${RR_I2yy}"
+        I3xx="${RR_I3xx}" I3yy="${RR_I3yy}" I3zz="${RR_I3yy}"
+        I4xx="${RR_I4xx}" I4yy="${RR_I4yy}" I4zz="${RR_I4yy}" />
 </robot>

Commit message: Moved gait generation related functionality to the gait_generation package. Generated pendulum power script for simple case testing

File: src/quadruped_description/xacro/leg.xacro (robot description, xacro)
@@ -63,4 +63,6 @@
             <child
                 link="${child}" />
+            <!-- <axis xyz="1 0 0" /> -->
+            <!-- <limits effort="0.0" velocity="0.0" lower="0.0" upper="0.0" /> -->
         </joint>
     </xacro:macro>

File: src/quadruped_description/xacro/quad_plugins.xacro (robot description, xacro)
@@ -5,4 +5,8 @@
         <uri>
             /workspace/install/quadruped_description/share/quadruped_description/urdf/quadruped.urdf</uri>
+        <plugin filename="libgz-sim-apply-joint-force-system"
+            name="gz::sim::v8::systems::ApplyJointForce">
+            <joint_name>z_trans_x_trans_joint</joint_name>
+        </plugin>
         <!-- Plugin for joint state publisher -->
         <plugin
@@ -10,4 +14,5 @@
             name="gz::sim::systems::JointStatePublisher">
             <topic>joint_states</topic>
+            <!-- Dynamic Joints -->
             <joint_name>FR_hip_joint</joint_name>
             <joint_name>FR_thigh_joint</joint_name>
@@ -35,5 +40,4 @@
             </plugin>
         </xacro:macro>
-        <!-- Plugin for joint controllers -->
         <!-- Explicitly Add All Joints -->
         <xacro:add_joint_controller joint_name="FR_hip_joint" Kp="100.0" Ki="0.1" Kd="10.0" />

File: src/quadruped_description/xacro/world_constraints.xacro (robot description, xacro)
@@ -1,4 +1,5 @@
 <?xml version="1.0" encoding="utf-8"?>
 <robot name="world_constraints" xmlns:xacro="http://www.ros.org/wiki/xacro">
+    <xacro:property name="world_constraints" value="${True}" />
     <!-- Generate Constraint using these joints -->
     <gazebo>
