Commit message: thesis version update

File: src/quadruped_description/xacro/const.xacro (robot description, xacro)
@@ -3,3 +3,4 @@
     <!-- Constants for robot dimensions -->
     <xacro:property name="PI" value="3.1415926535897931"/>
+    <xacro:property name="DAMPING_CONST" value="0.0"/>
 </robot>

File: src/quadruped_description/xacro/leg.xacro (robot description, xacro)
@@ -18,4 +18,5 @@
                     rpy="${PI/2} 0.0 ${PI/2}" />
             </xacro:if>
+            <dynamics damping="${DAMPING_CONST}" friction="0.0"/>
         </joint>
     </xacro:macro>
@@ -35,4 +36,5 @@
                     rpy="${-PI/2} 0 ${-PI/2}" />
             </xacro:if>
+            <dynamics damping="${DAMPING_CONST}" friction="0.0"/>
         </joint>
     </xacro:macro>
@@ -52,4 +54,5 @@
                     rpy="0.0 0.0 0.0" />
             </xacro:if>
+            <dynamics damping="${DAMPING_CONST}" friction="0.0"/>
         </joint>
     </xacro:macro>

File: src/quadruped_description/xacro/quad_plugins.xacro (robot description, xacro)
@@ -23,4 +23,5 @@
             <joint_name>RL_thigh_joint</joint_name>
             <joint_name>RL_calf_joint</joint_name>
+            <joint_name>z_trans_x_trans_joint</joint_name>
         </plugin>
         <!-- Macro for Joint Controllers -->
@@ -35,4 +36,6 @@
                 <d_gain>${Kd}</d_gain>
                 <torque_topic>/quadruped/${joint_name}_torque</torque_topic>
+                <cmd_max>33.5</cmd_max>
+                <cmd_min>-33.5</cmd_min>
             </plugin>
         </xacro:macro>
