Commit message: Configured for running simulations in series

File: src/quadruped_description/xacro/world_constraints.xacro (robot description, xacro)
@@ -33,5 +33,6 @@
             </axis>
         </joint>
-        <joint name="y_rotation" type="revolute">
+        <!-- <link name="x_rotation" /> -->
+        <joint name="x_rotation_joint" type="revolute">
             <parent>x_translation</parent>
             <child>base</child>
@@ -44,4 +45,15 @@
             </axis>
         </joint>
+        <!-- <joint name="y_rotation_joint" type="revolute">
+            <parent>x_rotation</parent>
+            <child>base</child>
+            <axis>
+                <xyz>0 1 0</xyz>
+                <limit>
+                    <lower>${-PI/75}</lower>
+                    <upper>${PI/75}</upper>
+                </limit>
+            </axis>
+        </joint> -->
     </gazebo>
 </robot>
