Commit message: Added planar constraints to gazebo simulation. fixed bugs in gait loader

File: src/quadruped_description/xacro/quad_plugins.xacro (robot description, xacro)
@@ -3,6 +3,6 @@
     <include>
         <!-- Robot URDF -->
-        <uri>/workspace/install/quadruped_description/share/quadruped_description/urdf/quadruped.urdf</uri>
-        <!-- <uri>/workspace/src/robot_descriptions/a1_description/urdf/a1.urdf</uri> -->
+        <uri>
+            /workspace/install/quadruped_description/share/quadruped_description/urdf/quadruped.urdf</uri>
         <!-- Plugin for joint state publisher -->
         <plugin

File: src/quadruped_description/xacro/quadruped.xacro (robot description, xacro)
@@ -1,4 +1,30 @@
 <?xml version="1.0" encoding="utf-8"?>
 <robot name="quadruped" xmlns:xacro="http://www.ros.org/wiki/xacro">
+    <!-- Generate Planar Constraint using these joints -->
+    <gazebo>
+        <link name="z_movement" />
+        <joint name="world_z_joint" type="prismatic">
+            <parent>world</parent>
+            <child>z_movement</child>
+            <axis>
+                <xyz>0 0 1</xyz>
+                <limit>
+                    <lower>-10</lower>
+                    <upper>10</upper>
+                </limit>
+            </axis>
+        </joint>
+        <joint name="x_movement" type="prismatic">
+            <parent>z_movement</parent>
+            <child>base</child>
+            <axis>
+                <xyz>1 0 0</xyz>
+                <limit>
+                    <lower>-10</lower>
+                    <upper>100</upper>
+                </limit>
+            </axis>
+        </joint>
+    </gazebo>
     <!-- Define colors for links -->
     <xacro:include
@@ -12,9 +38,9 @@
     <xacro:base_link
         name="base" L_x="${base_Lx}" L_y="${base_Ly}" L_z="${base_Lz}" mass="${base_m}"
-        inertial_link="False" Ixx="${base_Ixx}" Iyy="${base_Iyy}" Izz="${base_Izz}"/>
+        inertial_link="False" Ixx="${base_Ixx}" Iyy="${base_Iyy}" Izz="${base_Izz}" />
     <!-- Insert dummy link to carry inertia values for base link -->
     <xacro:base_link
         name="base_inertia" L_x="${base_Lx}" L_y="${base_Ly}" L_z="${base_Lz}" mass="${base_m}"
-        inertial_link="True" Ixx="${base_Ixx}" Iyy="${base_Iyy}" Izz="${base_Izz}"/>
+        inertial_link="True" Ixx="${base_Ixx}" Iyy="${base_Iyy}" Izz="${base_Izz}" />
     <xacro:fixed_joint name="inertial_base_joint" parent="base" child="base_inertia" length="0.0" />
     <xacro:leg leg_name="FR" right="True"

Commit message: Augmented jointpositioncontroller to print instantaneous applied torque

File: src/quadruped_description/xacro/quad_plugins.xacro (robot description, xacro)
@@ -5,8 +5,4 @@
         <uri>
             /workspace/install/quadruped_description/share/quadruped_description/urdf/quadruped.urdf</uri>
-        <plugin filename="libgz-sim-apply-joint-force-system"
-            name="gz::sim::v8::systems::ApplyJointForce">
-            <joint_name>z_trans_x_trans_joint</joint_name>
-        </plugin>
         <!-- Plugin for joint state publisher -->
         <plugin
@@ -29,5 +25,5 @@
         </plugin>
         <!-- Macro for Joint Controllers -->
-        <xacro:macro name="add_joint_controller" params="joint_name Kp Ki Kd">
+        <!-- <xacro:macro name="add_joint_controller" params="joint_name">
             <plugin
                 filename="gz-sim-joint-position-controller-system"
@@ -39,18 +35,28 @@
                 <d_gain>1</d_gain>
             </plugin>
+        </xacro:macro> -->
+        <xacro:macro name="add_joint_controller" params="joint_name">
+            <plugin filename="libgz-sim-apply-joint-force-system"
+                name="gz::sim::v8::systems::ApplyJointForce">
+                <joint_name>${joint_name}</joint_name>
+            </plugin>
         </xacro:macro>
+        <plugin filename="libgz-sim-apply-joint-force-system"
+            name="gz::sim::v8::systems::ApplyJointForce">
+            <joint_name>z_trans_x_trans_joint</joint_name>
+        </plugin>
         <!-- Explicitly Add All Joints -->
-        <xacro:add_joint_controller joint_name="FR_hip_joint" Kp="100.0" Ki="0.1" Kd="10.0" />
-        <xacro:add_joint_controller joint_name="FR_thigh_joint" Kp="100.0" Ki="0.1" Kd="10.0" />
-        <xacro:add_joint_controller joint_name="FR_calf_joint" Kp="100.0" Ki="0.1" Kd="10.0" />
-        <xacro:add_joint_controller joint_name="FL_hip_joint" Kp="100.0" Ki="0.1" Kd="10.0" />
-        <xacro:add_joint_controller joint_name="FL_thigh_joint" Kp="100.0" Ki="0.1" Kd="10.0" />
-        <xacro:add_joint_controller joint_name="FL_calf_joint" Kp="100.0" Ki="0.1" Kd="10.0" />
-        <xacro:add_joint_controller joint_name="RR_hip_joint" Kp="100.0" Ki="0.1" Kd="10.0" />
-        <xacro:add_joint_controller joint_name="RR_thigh_joint" Kp="100.0" Ki="0.1" Kd="10.0" />
-        <xacro:add_joint_controller joint_name="RR_calf_joint" Kp="100.0" Ki="0.1" Kd="10.0" />
-        <xacro:add_joint_controller joint_name="RL_hip_joint" Kp="100.0" Ki="0.1" Kd="10.0" />
-        <xacro:add_joint_controller joint_name="RL_thigh_joint" Kp="100.0" Ki="0.1" Kd="10.0" />
-        <xacro:add_joint_controller joint_name="RL_calf_joint" Kp="100.0" Ki="0.1" Kd="10.0" />
+        <xacro:add_joint_controller joint_name="FR_hip_joint" />
+        <xacro:add_joint_controller joint_name="FR_thigh_joint" />
+        <xacro:add_joint_controller joint_name="FR_calf_joint" />
+        <xacro:add_joint_controller joint_name="FL_hip_joint" />
+        <xacro:add_joint_controller joint_name="FL_thigh_joint" />
+        <xacro:add_joint_controller joint_name="FL_calf_joint" />
+        <xacro:add_joint_controller joint_name="RR_hip_joint" />
+        <xacro:add_joint_controller joint_name="RR_thigh_joint" />
+        <xacro:add_joint_controller joint_name="RR_calf_joint" />
+        <xacro:add_joint_controller joint_name="RL_hip_joint" />
+        <xacro:add_joint_controller joint_name="RL_thigh_joint" />
+        <xacro:add_joint_controller joint_name="RL_calf_joint" />
     </include>
 </sdf>

Commit message: Added gazebo plugin functionallity to publish joint torques

File: src/quadruped_description/xacro/quad_plugins.xacro (robot description, xacro)
@@ -25,8 +25,8 @@
         </plugin>
         <!-- Macro for Joint Controllers -->
-        <!-- <xacro:macro name="add_joint_controller" params="joint_name">
+        <xacro:macro name="add_joint_controller" params="joint_name">
             <plugin
-                filename="gz-sim-joint-position-controller-system"
-                name="gz::sim::systems::JointPositionController">
+                filename="libJointPositionControllerTorquePublisher.so"
+                name="quadruped_gazebo::JointPositionControllerTorquePublisher">
                 <joint_name>${joint_name}</joint_name>
                 <topic>quadruped/cmd_${joint_name}</topic>
@@ -34,10 +34,5 @@
                 <i_gain>0</i_gain>
                 <d_gain>1</d_gain>
-            </plugin>
-        </xacro:macro> -->
-        <xacro:macro name="add_joint_controller" params="joint_name">
-            <plugin filename="libgz-sim-apply-joint-force-system"
-                name="gz::sim::v8::systems::ApplyJointForce">
-                <joint_name>${joint_name}</joint_name>
+                <torque_topic>/quadruped/${joint_name}_torque</torque_topic>
             </plugin>
         </xacro:macro>

Commit message: Updated plot generation, Removed derivitive kick, tuned PID gains

File: src/quadruped_description/xacro/quad_plugins.xacro (robot description, xacro)
@@ -25,5 +25,5 @@
         </plugin>
         <!-- Macro for Joint Controllers -->
-        <xacro:macro name="add_joint_controller" params="joint_name">
+        <xacro:macro name="add_joint_controller" params="joint_name Kp Ki Kd">
             <plugin
                 filename="libJointPositionControllerTorquePublisher.so"
@@ -31,7 +31,7 @@
                 <joint_name>${joint_name}</joint_name>
                 <topic>quadruped/cmd_${joint_name}</topic>
-                <p_gain>20</p_gain>
-                <i_gain>0</i_gain>
-                <d_gain>1</d_gain>
+                <p_gain>${Kp}</p_gain>
+                <i_gain>${Ki}</i_gain>
+                <d_gain>${Kd}</d_gain>
                 <torque_topic>/quadruped/${joint_name}_torque</torque_topic>
             </plugin>
@@ -41,17 +41,29 @@
             <joint_name>z_trans_x_trans_joint</joint_name>
         </plugin>
+        <!-- Hip PID Gains -->
+        <xacro:property name="hip_Kp" value="100.0" />
+        <xacro:property name="hip_Ki" value="0.0" />
+        <xacro:property name="hip_Kd" value="2.0" />
+        <!-- Thigh PID Gains -->
+        <xacro:property name="thigh_Kp" value="250.0" />
+        <xacro:property name="thigh_Ki" value="0.0" />
+        <xacro:property name="thigh_Kd" value="2.5" />
+        <!-- Calf PID Gains -->
+        <xacro:property name="calf_Kp" value="350.0" />
+        <xacro:property name="calf_Ki" value="0.0" />
+        <xacro:property name="calf_Kd" value="3.5" />
         <!-- Explicitly Add All Joints -->
-        <xacro:add_joint_controller joint_name="FR_hip_joint" />
-        <xacro:add_joint_controller joint_name="FR_thigh_joint" />
-        <xacro:add_joint_controller joint_name="FR_calf_joint" />
-        <xacro:add_joint_controller joint_name="FL_hip_joint" />
-        <xacro:add_joint_controller joint_name="FL_thigh_joint" />
-        <xacro:add_joint_controller joint_name="FL_calf_joint" />
-        <xacro:add_joint_controller joint_name="RR_hip_joint" />
-        <xacro:add_joint_controller joint_name="RR_thigh_joint" />
-        <xacro:add_joint_controller joint_name="RR_calf_joint" />
-        <xacro:add_joint_controller joint_name="RL_hip_joint" />
-        <xacro:add_joint_controller joint_name="RL_thigh_joint" />
-        <xacro:add_joint_controller joint_name="RL_calf_joint" />
+        <xacro:add_joint_controller joint_name="FR_hip_joint" Kp="${hip_Kp}" Ki="${hip_Ki}" Kd="${hip_Kd}" />
+        <xacro:add_joint_controller joint_name="FR_thigh_joint" Kp="${thigh_Kp}" Ki="${thigh_Ki}" Kd="${thigh_Kd}" />
+        <xacro:add_joint_controller joint_name="FR_calf_joint" Kp="${calf_Kp}" Ki="${calf_Ki}" Kd="${calf_Kd}" />
+        <xacro:add_joint_controller joint_name="FL_hip_joint" Kp="${hip_Kp}" Ki="${hip_Ki}" Kd="${hip_Kd}" />
+        <xacro:add_joint_controller joint_name="FL_thigh_joint" Kp="${thigh_Kp}" Ki="${thigh_Ki}" Kd="${thigh_Kd}" />
+        <xacro:add_joint_controller joint_name="FL_calf_joint" Kp="${calf_Kp}" Ki="${calf_Ki}" Kd="${calf_Kd}" />
+        <xacro:add_joint_controller joint_name="RR_hip_joint" Kp="${hip_Kp}" Ki="${hip_Ki}" Kd="${hip_Kd}" />
+        <xacro:add_joint_controller joint_name="RR_thigh_joint" Kp="${thigh_Kp}" Ki="${thigh_Ki}" Kd="${thigh_Kd}" />
+        <xacro:add_joint_controller joint_name="RR_calf_joint" Kp="${calf_Kp}" Ki="${calf_Ki}" Kd="${calf_Kd}" />
+        <xacro:add_joint_controller joint_name="RL_hip_joint" Kp="${hip_Kp}" Ki="${hip_Ki}" Kd="${hip_Kd}" />
+        <xacro:add_joint_controller joint_name="RL_thigh_joint" Kp="${thigh_Kp}" Ki="${thigh_Ki}" Kd="${thigh_Kd}" />
+        <xacro:add_joint_controller joint_name="RL_calf_joint" Kp="${calf_Kp}" Ki="${calf_Ki}" Kd="${calf_Kd}" />
     </include>
 </sdf>

Commit message: Ran parameter variation simulations. Logged data

File: src/quadruped_description/xacro/quad_plugins.xacro (robot description, xacro)
@@ -45,5 +45,10 @@
         </plugin>
         <!-- Hip PID Gains -->
-        <xacro:property name="hip_Kp" value="100.0" />
+        <!-- originial -->
+        <!-- <xacro:property name="hip_Kp" value="100.0" />
+        <xacro:property name="hip_Ki" value="0.0" />
+        <xacro:property name="hip_Kd" value="2.0" />
+         -->
+        <xacro:property name="hip_Kp" value="10.0" />
         <xacro:property name="hip_Ki" value="0.0" />
         <xacro:property name="hip_Kd" value="2.0" />
@@ -53,7 +58,7 @@
         <xacro:property name="thigh_Kd" value="2.5" />
         <!-- Calf PID Gains -->
-        <xacro:property name="calf_Kp" value="350.0" />
+        <xacro:property name="calf_Kp" value="250.0" />
         <xacro:property name="calf_Ki" value="0.0" />
-        <xacro:property name="calf_Kd" value="3.5" />
+        <xacro:property name="calf_Kd" value="2.5" />
         <!-- Explicitly Add All Joints -->
         <xacro:add_joint_controller joint_name="FR_hip_joint" Kp="${hip_Kp}" Ki="${hip_Ki}" Kd="${hip_Kd}" />

File: src/quadruped_description/xacro/world_constraints.xacro (robot description, xacro)
@@ -34,7 +34,7 @@
         </joint>
         <!-- <link name="x_rotation" /> -->
-        <joint name="x_rotation_joint" type="revolute">
+        <!-- <joint name="x_rotation_joint" type="revolute">
             <parent>x_translation</parent>
-            <child>base</child>
+            <child>x_rotation</child>
             <axis>
                 <xyz>1 0 0</xyz>
@@ -44,16 +44,16 @@
                 </limit>
             </axis>
-        </joint>
-        <!-- <joint name="y_rotation_joint" type="revolute">
-            <parent>x_rotation</parent>
+        </joint> -->
+        <joint name="y_rotation_joint" type="revolute">
+            <parent>x_translation</parent>
             <child>base</child>
             <axis>
                 <xyz>0 1 0</xyz>
                 <limit>
-                    <lower>${-PI/75}</lower>
-                    <upper>${PI/75}</upper>
+                    <lower>${-PI/12}</lower>
+                    <upper>${PI/12}</upper>
                 </limit>
             </axis>
-        </joint> -->
+        </joint>
     </gazebo>
 </robot>
